File: kicad/stm32_hotswap_chiffre.kicad_pcb (KiCad board)
At the start: 2 copper layers, 227.3 x 85 mm, 110 parts, among them J1 USB_C_Receptacle_USB2.0, J101 Conn_01x03_Female, J2 OLED I2C, J3 SW_DEBUG, SW1 SW_Push, SW10 SW_Push, SW11 SW_Push, SW12 SW_Push, SW13 SW_Push, SW14 SW_Push, SW15 SW_Push, SW16 SW_Push, SW17 SW_Push, SW18 SW_Push, SW19 SW_Push, SW2 SW_Push, SW20 SW_Push, SW21 SW_Push, SW22 SW_Push, SW23 SW_Push, SW24 SW_Push, SW25 SW_Push, SW26 SW_Push, SW27 SW_Push, SW28 SW_Push, SW29 SW_Push, SW3 SW_Push, SW30 SW_Push, SW31 SW_Push, SW32 SW_Push, SW33 SW_Push, SW34 SW_Push, SW35 SW_Push, SW36 Rotary_Encoder_Switch, SW37 SKQGABE010, SW38 SKQGABE010, SW4 SW_Push, SW5 SW_Push, SW6 SW_Push, SW7 SW_Push, SW8 SW_Push, SW9 SW_Push, U1 XC6206PxxxMR-Regulator_Linear, U2 STM32F072CBT6, U3 USBLC6-2SC6

Commit message: cleaning up pcb
Parts:
- added C11: DNP, Capacitor_SMD:C_0402_1005Metric, B.Cu at (142.2, 73.3)
- added FB1: FerriteBead_Small, Inductor_SMD:L_0805_2012Metric, B.Cu at (147.9, 73.6)
- R1, R2, R3, R4, R5, R6: footprint Resistor_SMD:R_0603_1608Metric -> Resistor_SMD:R_0402_1005Metric
- moved C2 10.6 mm to (154.9, 76.2), turned to 180 degrees
- moved R1 10.4 mm to (142.8, 70.9)
- moved C12 6.67 mm to (149.7, 72.3)
- moved U1 5.30 mm to (151.9, 74.4), turned to 180 degrees
- moved U3 3.27 mm to (145.3, 71.8)
- moved R2 3.16 mm to (151.6, 72.3), turned to 180 degrees
- moved R4 1.37 mm to (152.7, 124.5), turned to -45 degrees
- moved R3 1.00 mm to (153.5, 123.8), turned to 135 degrees
- moved F1 0.74 mm to (149.3, 70.4)
- moved C1 0.28 mm to (149.4, 74.5), turned to -90 degrees
- renumbered C8 to C13, C11 to C7, C7 to C8
Connections:
- net CC1 renamed Net-(J1-CC1)
- net CC2 renamed Net-(J1-CC2)
- C12 pad 1: +5V -> /VBUS_fused
- F1 pad 2: +5V -> /VBUS_fused
- U2 pad 32: USB_D_N -> D_N
- U2 pad 33: USB_D_P -> D_P
- U3 pad 1: USB_D_P -> D_P
- U3 pad 3: USB_D_N -> D_N
- U3 pad 5: +5V -> /VBUS_fused
Routing:
- net USB_D_N: track 71.1 -> 6.35 mm, vias 2 -> 0
- net D_N: track 0.00 -> 61.2 mm
- net D_P: track 0.00 -> 61.1 mm
- net USB_D_P: track 65.3 -> 6.25 mm
- net Net-(J1-CC1): track 17.4 -> 4.06 mm, vias 2 -> 0
- net /VBUS_fused: track 0.00 -> 7.46 mm
- net Net-(J1-CC2): track 9.80 -> 5.58 mm
- net +3V3: track 142.7 -> 138.9 mm, vias 8 -> 10
- net GND: track 54.4 -> 50.8 mm, vias 59 -> 79
- net SDA: track 40.6 -> 38.3 mm, vias 0 -> 1
- net +5V: track 603.8 -> 605.7 mm, vias 17 -> 13
- net Net-(R3-Pad1): track 29.4 -> 30.4 mm, vias 2 -> 3
- net Net-(D35-K): track 29.1 -> 28.2 mm
- net SWCLK: track 22.0 -> 22.7 mm
- net EncB: track 41.9 -> 42.6 mm
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Other:
- board text added: "Le Chiffre STM32 v0.2"
- board text removed: "D100"
- board text removed: "Le Chiffre STM32 v0.1 by sporkus"

Commit message: v0.2
Parts:
- removed the C11 at (142.2, 73.3)
- removed FB1: FerriteBead_Small, Inductor_SMD:L_0805_2012Metric
- removed J3: SW_DEBUG, Connector_PinHeader_2.54mm:PinHeader_1x04_P2.54mm_Vertical
- removed the R3 at (153.5, 123.8)
- removed the SW37 at (146.6, 112.8)
- added L1: 60R@100MHz, Inductor_SMD:L_1206_3216Metric, B.Cu at (141.3, 72.5)
- SW36: footprint Keebio-Parts:RotaryEncoder_EC11 -> modified_footrprints:RotaryEncoder_EC11_no_mp
- U2: renamed from U3; value USBLC6-2SC6 -> PRTR5V0U2X; footprint Package_TO_SOT_SMD:SOT-23-6 -> Package_TO_SOT_SMD:SOT-143
- moved R3 19.2 mm to (150.6, 105.4), turned to -90 degrees
- moved C7 11.3 mm to (153.5, 124.0)
- moved D32 11.0 mm to (99.8, 125.4), turned to 83 degrees
- moved D33 10.8 mm to (179.3, 126.7), turned to 97 degrees
- moved C6 10.7 mm to (150.9, 116.2), turned to -90 degrees
- moved D35 10.4 mm to (151.8, 88.4)
- moved D31 9.59 mm to (68.3, 122.8), turned to 83 degrees
- moved C5 9.46 mm to (150.9, 119.2), turned to 90 degrees
- moved C3 9.01 mm to (149.1, 117.7), turned to 180 degrees
- moved D30 8.84 mm to (238.3, 114.9)
- moved C4 8.63 mm to (152.2, 124.6), turned to 90 degrees
- moved D34 7.78 mm to (209.8, 124.2), turned to 97 degrees
- moved C10 6.01 mm to (141.8, 92.3), turned to -90 degrees
- moved U1 4.93 mm to (146.5, 123.3), turned to 180 degrees
- moved C2 4.44 mm to (140.8, 120.8), turned to -90 degrees
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- renumbered C3 to C1, C1 to C11, C2 to C12, C4 to C2, C5 to C3, C6 to C4, C7 to C5, C8 to C6, C13 to C7, C12 to C8, R4 to R3, R5 to R4, R6 to R5, SW38 to SW37, U2 to U1, U1 to U3
Connections:
- C7 pad 1: GND -> NRST
- C7 pad 2: NRST -> GND
- C8 pad 1: /VBUS_fused -> +5V
- C8 pad 2: GND -> GNDPWR
- F1 pad 2: /VBUS_fused -> +5V
- J1 pad A1: GND -> GNDPWR
- J1 pad A12: GND -> GNDPWR
- J1 pad A6: USB_D_P -> D_P
- J1 pad A7: USB_D_N -> D_N
- J1 pad B1: GND -> GNDPWR
- J1 pad B12: GND -> GNDPWR
- J1 pad B6: USB_D_P -> D_P
- J1 pad B7: USB_D_N -> D_N
- J1 pad S1: GND -> GNDPWR
- R1 pad 1: GND -> GNDPWR
- R2 pad 1: GND -> GNDPWR
- SW37 pad 2: Net-(R3-Pad1) -> BOOT0
- U1 pad 34: SWDIO -> unconnected-(U1-PA13-Pad34)
- U1 pad 37: SWCLK -> unconnected-(U1-PA14-Pad37)
- U2 pad 1: D_P -> GNDPWR
- U2 pad 2: GND -> D_N
- U2 pad 3: D_N -> D_P
- U2 pad 4: USB_D_N -> +5V
Routing:
- net +5V: track 605.7 -> 730.0 mm, vias 13 -> 18
- net row0: track 380.2 -> 303.1 mm, vias 15 -> 6
- net row3: track 249.0 -> 200.4 mm, vias 2 -> 4
- net Net-(R3-Pad1): track 30.4 -> 0.00 mm, vias 3 -> 0
- net row1: track 312.0 -> 282.8 mm, vias 14 -> 6
- net +3V3: track 138.9 -> 111.0 mm, vias 10 -> 8
- net row2: track 252.0 -> 225.0 mm, vias 11 -> 2
- net SWCLK: track 22.7 -> 0.00 mm
- net BOOT0: track 3.75 -> 26.3 mm, vias 0 -> 2
- net SWDIO: track 21.1 -> 0.00 mm
- net col7: track 162.2 -> 144.0 mm
- net col8: track 157.3 -> 139.4 mm, vias 2 -> 1
- net col9: track 178.6 -> 161.7 mm, vias 1 -> 0
- net col6: track 137.4 -> 121.5 mm
- net Net-(D108-DOUT): track 39.7 -> 55.2 mm, vias 0 -> 2
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- added copper zone on B.Cu, net GNDPWR
- added copper zone on F.Cu, net GNDPWR
Other:
- board text added: "Le Chiffre 32 v0.2 by sporkus"
- board text removed: "Le Chiffre STM32 v0.2"
- board text removed: "RST"
- board text removed: "optional"
- board text removed: "swclk"
- board text removed: "swdio"

Commit message: v0.2 release
Parts:
- moved C7 0.33 mm to (153.2, 124.2)
Connections:
- C8 pad 2: GNDPWR -> GND
- J1 pad A1: GNDPWR -> GND
- J1 pad A12: GNDPWR -> GND
- J1 pad B1: GNDPWR -> GND
- J1 pad B12: GNDPWR -> GND
- J1 pad S1: GNDPWR -> GND
- L1 pad 1: GNDPWR -> GND
- R1 pad 1: GNDPWR -> GND
- R2 pad 1: GNDPWR -> GND
Routing:
- net +5V: track 730.0 -> 649.0 mm, vias 18 -> 16
- net col7: track 144.0 -> 160.3 mm, vias 1 -> 0
- net col6: track 121.5 -> 137.7 mm
- net GNDPWR: track 13.6 -> 0.00 mm, vias 6 -> 0
- net col5: track 136.1 -> 148.3 mm, vias 4 -> 5
- net row0: track 303.1 -> 295.8 mm
- net row2: track 225.0 -> 231.3 mm, vias 2 -> 4
- net Net-(D101-DOUT): track 14.4 -> 20.3 mm
- net row1: track 282.8 -> 277.3 mm
- net GND: track 42.7 -> 48.0 mm, vias 120 -> 128
- net Net-(D105-DOUT): track 58.9 -> 55.4 mm
- net col3: track 96.1 -> 99.5 mm, vias 1 -> 0
- net Net-(D110-DOUT): track 86.1 -> 83.4 mm
- net Net-(D111-DOUT): track 90.8 -> 93.3 mm
- net col2: track 142.3 -> 139.9 mm, vias 1 -> 0
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- removed copper zone on B.Cu, net GNDPWR
- removed copper zone on F.Cu, net GNDPWR
