File: kicad/key_matrix.kicad_sch (KiCad schematic)
At the start: 71 parts, among them SW1 SW_Push, SW10 SW_Push, SW11 SW_Push, SW12 SW_Push, SW13 SW_Push, SW14 SW_Push, SW15 SW_Push, SW16 SW_Push, SW17 SW_Push, SW18 SW_Push, SW19 SW_Push, SW2 SW_Push, SW20 SW_Push, SW21 SW_Push, SW22 SW_Push, SW23 SW_Push, SW24 SW_Push, SW25 SW_Push, SW26 SW_Push, SW27 SW_Push, SW28 SW_Push, SW29 SW_Push, SW3 SW_Push, SW30 SW_Push, SW31 SW_Push, SW32 SW_Push, SW33 SW_Push, SW34 SW_Push, SW35 SW_Push, SW36 Rotary_Encoder_Switch, SW4 SW_Push, SW5 SW_Push, SW6 SW_Push, SW7 SW_Push, SW8 SW_Push, SW9 SW_Push

Commit message: bom
Parts:
- SW1: now left out of the parts list
Changed lines of the file:
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@@
   )
   (symbol (lib_id "Switch:SW_Push") (at 66.04 52.07 0) (unit 1)
-    (in_bom yes) (on_board yes) (dnp no)
+    (in_bom no) (on_board yes) (dnp no)
     (property "Reference" "SW1" (at 66.04 44.831 0)
       (effects (font (size 1.27 1.27)))

Commit message: more bom work
Parts:
- D1, D10, D11, D12, D13, D14, D15, D16, D17, D18, D19, D2, D20, D21, D22, D23, D24, D25, D26, D27, D28, D29, D3, D30, D31, D32, D33, D34, D35, D4, D5, D6, D7, D8, D9: JlcRotOffset (none) -> 0
Changed lines of the file:
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@@
+      (effects (font (size 1.27 1.27)) hide)
+    )
+    (property "JlcRotOffset" "0" (at 199.39 74.93 0)
       (effects (font (size 1.27 1.27)) hide)
     )
@@
       (effects (font (size 1.27 1.27)) hide)
     )
+    (property "JlcRotOffset" "0" (at 102.87 74.93 0)
+      (effects (font (size 1.27 1.27)) hide)
+    )
     (pin "1")
     (pin "2")
@@
       (effects (font (size 1.27 1.27)) hide)
     )
+    (property "JlcRotOffset" "0" (at 171.45 113.03 0)
+      (effects (font (size 1.27 1.27)) hide)
+    )
     (pin "1")
     (pin "2")
@@
       (effects (font (size 1.27 1.27)) hide)
     )
+    (property "JlcRotOffset" "0" (at 62.23 140.97 0)
+      (effects (font (size 1.27 1.27)) hide)
+    )
     (pin "1")
     (pin "2")
@@
       (effects (font (size 1.27 1.27)) hide)
     )
+    (property "JlcRotOffset" "0" (at 116.84 55.88 0)
+      (effects (font (size 1.27 1.27)) hide)
+    )
     (pin "1")
     (pin "2")
@@
       (effects (font (size 1.27 1.27)) hide)
     )
+    (property "JlcRotOffset" "0" (at 88.9 93.98 0)
+      (effects (font (size 1.27 1.27)) hide)
+    )
     (pin "1")
     (pin "2")
@@
       (effects (font (size 1.27 1.27)) hide)
     )
+    (property "JlcRotOffset" "0" (at 74.93 74.93 0)
+      (effects (font (size 1.27 1.27)) hide)
+    )
     (pin "1")
     (pin "2")
@@
       (effects (font (size 1.27 1.27)) hide)
     )
+    (property "JlcRotOffset" "0" (at 171.45 93.98 0)
+      (effects (font (size 1.27 1.27)) hide)
+    )
     (pin "1")
     (pin "2")
@@
       (effects (font (size 1.27 1.27)) hide)
     )
+    (property "JlcRotOffset" "0" (at 143.51 113.03 0)
+      (effects (font (size 1.27 1.27)) hide)
+    )
     (pin "1")
     (pin "2")
@@
     )
     (property "Datasheet" "https://assets.nexperia.com/documents/data-sheet/1N4148_1N4448.pdf" (at 143.51 93.98 0)
+      (effects (font (size 1.27 1.27)) hide)
+    )
+    (property "JlcRotOffset" "0" (at 143.51 93.98 0)
       (effects (font (size 1.27 1.27)) hide)
     )
@@
       (effects (font (size 1.27 1.27)) hide)
     )
+    (property "JlcRotOffset" "0" (at 88.9 74.93 0)
+      (effects (font (size 1.27 1.27)) hide)
+    )
     (pin "1")
     (pin "2")
@@
       (effects (font (size 1.27 1.27)) hide)
     )
+    (property "JlcRotOffset" "0" (at 116.84 113.03 0)
+      (effects (font (size 1.27 1.27)) hide)
+    )
     (pin "1")
     (pin "2")
@@
       (effects (font (size 1.27 1.27)) hide)
     )
+    (property "JlcRotOffset" "0" (at 157.48 55.88 0)
+      (effects (font (size 1.27 1.27)) hide)
+    )
     (pin "1")
     (pin "2")
@@
       (effects (font (size 1.27 1.27)) hide)
     )
+    (property "JlcRotOffset" "0" (at 102.87 93.98 0)
+      (effects (font (size 1.27 1.27)) hide)
+    )
     (pin "1")
     (pin "2")
@@
       (effects (font (size 1.27 1.27)) hide)
     )
+    (property "JlcRotOffset" "0" (at 74.93 93.98 0)
+      (effects (font (size 1.27 1.27)) hide)
+    )
     (pin "1")
     (pin "2")
@@
       (effects (font (size 1.27 1.27)) hide)
     )
+    (property "JlcRotOffset" "0" (at 157.48 74.93 0)
+      (effects (font (size 1.27 1.27)) hide)
+    )
     (pin "1")
     (pin "2")
@@
       (effects (font (size 1.27 1.27)) hide)
     )
+    (property "JlcRotOffset" "0" (at 143.51 55.88 0)
+      (effects (font (size 1.27 1.27)) hide)
+    )
     (pin "1")
     (pin "2")
@@
       (effects (font (size 1.27 1.27)) hide)
     )
+    (property "JlcRotOffset" "0" (at 88.9 55.88 0)
+      (effects (font (size 1.27 1.27)) hide)
+    )
     (pin "1")
     (pin "2")
@@
       (effects (font (size 1.27 1.27)) hide)
     )
+    (property "JlcRotOffset" "0" (at 88.9 113.03 0)
+      (effects (font (size 1.27 1.27)) hide)
+    )
     (pin "1")
     (pin "2")
@@
     )
     (property "Datasheet" "https://assets.nexperia.com/documents/data-sheet/1N4148_1N4448.pdf" (at 199.39 93.98 0)
+      (effects (font (size 1.27 1.27)) hide)
+    )
+    (property "JlcRotOffset" "0" (at 199.39 93.98 0)
       (effects (font (size 1.27 1.27)) hide)
     )
@@
       (effects (font (size 1.27 1.27)) hide)
     )
+    (property "JlcRotOffset" "0" (at 143.51 74.93 0)
+      (effects (font (size 1.27 1.27)) hide)
+    )
     (pin "1")
     (pin "2")
@@
       (effects (font (size 1.27 1.27)) hide)
     )
+    (property "JlcRotOffset" "0" (at 74.93 55.88 0)
+      (effects (font (size 1.27 1.27)) hide)
+    )
     (pin "1")
     (pin "2")
@@
       (effects (font (size 1.27 1.27)) hide)
     )
+    (property "JlcRotOffset" "0" (at 199.39 55.88 0)
+      (effects (font (size 1.27 1.27)) hide)
+    )
     (pin "1")
     (pin "2")
@@
       (effects (font (size 1.27 1.27)) hide)
     )
+    (property "JlcRotOffset" "0" (at 116.84 74.93 0)
+      (effects (font (size 1.27 1.27)) hide)
+    )
     (pin "1")
     (pin "2")
@@
       (effects (font (size 1.27 1.27)) hide)
     )
+    (property "JlcRotOffset" "0" (at 171.45 74.93 0)
+      (effects (font (size 1.27 1.27)) hide)
+    )
     (pin "1")
     (pin "2")
@@
       (effects (font (size 1.27 1.27)) hide)
     )
+    (property "JlcRotOffset" "0" (at 171.45 55.88 0)
+      (effects (font (size 1.27 1.27)) hide)
+    )
     (pin "1")
     (pin "2")
@@
       (effects (font (size 1.27 1.27)) hide)
     )
+    (property "JlcRotOffset" "0" (at 60.96 93.98 0)
+      (effects (font (size 1.27 1.27)) hide)
+    )
     (pin "1")
     (pin "2")
@@
       (effects (font (size 1.27 1.27)) hide)
     )
+    (property "JlcRotOffset" "0" (at 60.96 55.88 0)
+      (effects (font (size 1.27 1.27)) hide)
+    )
     (pin "1")
     (pin "2")
@@
       (effects (font (size 1.27 1.27)) hide)
     )
+    (property "JlcRotOffset" "0" (at 157.48 93.98 0)
+      (effects (font (size 1.27 1.27)) hide)
+    )
     (pin "1")
     (pin "2")
@@
       (effects (font (size 1.27 1.27)) hide)
     )
+    (property "JlcRotOffset" "0" (at 116.84 93.98 0)
+      (effects (font (size 1.27 1.27)) hide)
+    )
     (pin "1")
     (pin "2")
@@
       (effects (font (size 1.27 1.27)) hide)
     )
+    (property "JlcRotOffset" "0" (at 185.42 55.88 0)
+      (effects (font (size 1.27 1.27)) hide)
+    )
     (pin "1")
     (pin "2")
@@
       (effects (font (size 1.27 1.27)) hide)
     )
+    (property "JlcRotOffset" "0" (at 185.42 74.93 0)
+      (effects (font (size 1.27 1.27)) hide)
+    )
     (pin "1")
     (pin "2")
@@
       (effects (font (size 1.27 1.27)) hide)
     )
+    (property "JlcRotOffset" "0" (at 102.87 55.88 0)
+      (effects (font (size 1.27 1.27)) hide)
+    )
     (pin "1")
     (pin "2")
@@
       (effects (font (size 1.27 1.27)) hide)
     )
+    (property "JlcRotOffset" "0" (at 60.96 74.93 0)
+      (effects (font (size 1.27 1.27)) hide)
+    )
     (pin "1")
     (pin "2")
@@
       (effects (font (size 1.27 1.27)) hide)
     )
+    (property "JlcRotOffset" "0" (at 185.42 93.98 0)
+      (effects (font (size 1.27 1.27)) hide)
+    )

Commit message: encoder debounce caps + verified CPL
Parts:
- added C18, C19: 100nF, Capacitor_SMD:C_0402_1005Metric, symbol Device:C
- D1, D11, D12, D13, D14, D15, D2, D21, D22, D23, D24, D25, D3, D31, D32, D4, D5: JlcRotOffset 0 -> 14
- D10, D16, D17, D18, D19, D20, D26, D27, D28, D29, D30, D33, D34, D6, D7, D8, D9: JlcRotOffset 0 -> -14
Connections:
- net EncA: now also C19.1
- net EncB: now also C18.1
- net GND: now also C18.2, C19.2

Commit message: v0.2
Parts:
- SW1: now in the parts list
- SW36: now left out of the parts list
Other:
- company: (none) -> sporkus
- title: (none) -> Hotswap Chiffre
- moved on the sheet: C18, C19, D10, D16, D17, D18, D19, D20, D26, D27, D28, D29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

Commit message: adding front LED bypass jumper
Parts:
- SW36: footprint Keebio-Parts:RotaryEncoder_EC11 -> modified_footrprints:RotaryEncoder_EC11_no_mp
Changed lines of the file:
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@@
   (title_block
     (title "Hotswap Chiffre")
-    (date "2023-07-07")
-    (rev "0.2")
+    (date "2023-07-13")
+    (rev "0.2.1")
     (company "sporkus")
   )
@@
       (effects (font (size 1.27 1.27)))
     )
-    (property "Footprint" "Keebio-Parts:RotaryEncoder_EC11" (at 93.345 159.639 0)
-      (effects (font (size 1.27 1.27)) hide)
-    )
+    (property "Footprint" "modified_footrprints:RotaryEncoder_EC11_no_mp" (at 93.345 159.639 0)
+      (effects (font (size 1.27 1.27)) hide)
+    )

Commit message: change center switch footprint
Parts:
- SW35: footprint MX_hotswap_alps:MX-Hotswap-Alps-1U -> MX_Alps_Hybrid:MX-Alps-Hybrid-1U
Changed lines of the file:
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@@
       (effects (font (size 1.27 1.27)))
     )
-    (property "Footprint" "MX_hotswap_alps:MX-Hotswap-Alps-1U" (at 69.215 152.4 0)
+    (property "Footprint" "MX_Alps_Hybrid:MX-Alps-Hybrid-1U" (at 69.215 152.4 0)
       (effects (font (size 1.27 1.27)) hide)
     )
