File: kicad/rgb.kicad_sch (KiCad schematic)
At the start: 12 parts

Commit message: more bom work
Parts:
- D101, D102, D103, D104, D105, D106, D107, D108, D109, D110, D111: now left out of the parts list
Changed lines of the file:
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@@
   )
   (symbol (lib_id "LED:SK6812MINI") (at 97.79 58.42 0) (unit 1)
-    (in_bom yes) (on_board yes) (dnp no)
+    (in_bom no) (on_board yes) (dnp no)
     (property "Reference" "D102" (at 105.41 62.23 0)
       (effects (font (size 1.27 1.27)))
@@
   )
   (symbol (lib_id "LED:SK6812MINI") (at 90.17 86.36 0) (mirror y) (unit 1)
-    (in_bom yes) (on_board yes) (dnp no)
+    (in_bom no) (on_board yes) (dnp no)
     (property "Reference" "D110" (at 82.55 90.17 0)
       (effects (font (size 1.27 1.27)))
@@
   )
   (symbol (lib_id "LED:SK6812MINI") (at 72.39 86.36 0) (mirror y) (unit 1)
-    (in_bom yes) (on_board yes) (dnp no)
+    (in_bom no) (on_board yes) (dnp no)
     (property "Reference" "D111" (at 64.77 90.17 0)
       (effects (font (size 1.27 1.27)))
@@
   )
   (symbol (lib_id "LED:SK6812MINI") (at 107.95 86.36 0) (mirror y) (unit 1)
-    (in_bom yes) (on_board yes) (dnp no)
+    (in_bom no) (on_board yes) (dnp no)
     (property "Reference" "D109" (at 100.33 90.17 0)
       (effects (font (size 1.27 1.27)))
@@
   )
   (symbol (lib_id "LED:SK6812MINI") (at 115.57 58.42 0) (unit 1)
-    (in_bom yes) (on_board yes) (dnp no)
+    (in_bom no) (on_board yes) (dnp no)
     (property "Reference" "D103" (at 123.19 62.23 0)
       (effects (font (size 1.27 1.27)))
@@
   )
   (symbol (lib_id "LED:SK6812MINI") (at 143.51 86.36 0) (mirror y) (unit 1)
-    (in_bom yes) (on_board yes) (dnp no)
+    (in_bom no) (on_board yes) (dnp no)
     (property "Reference" "D107" (at 135.89 90.17 0)
       (effects (font (size 1.27 1.27)))
@@
   )
   (symbol (lib_id "LED:SK6812MINI") (at 133.35 58.42 0) (unit 1)
-    (in_bom yes) (on_board yes) (dnp no)
+    (in_bom no) (on_board yes) (dnp no)
     (property "Reference" "D104" (at 140.97 62.23 0)
       (effects (font (size 1.27 1.27)))
@@
   )
   (symbol (lib_id "LED:SK6812MINI") (at 125.73 86.36 0) (mirror y) (unit 1)
-    (in_bom yes) (on_board yes) (dnp no)
+    (in_bom no) (on_board yes) (dnp no)
     (property "Reference" "D108" (at 118.11 90.17 0)
       (effects (font (size 1.27 1.27)))
@@
   )
   (symbol (lib_id "LED:SK6812MINI") (at 80.01 58.42 0) (unit 1)
-    (in_bom yes) (on_board yes) (dnp no)
+    (in_bom no) (on_board yes) (dnp no)
     (property "Reference" "D101" (at 87.63 62.23 0)
       (effects (font (size 1.27 1.27)))
@@
   )
   (symbol (lib_id "LED:SK6812MINI") (at 161.29 86.36 0) (mirror y) (unit 1)
-    (in_bom yes) (on_board yes) (dnp no)
+    (in_bom no) (on_board yes) (dnp no)
     (property "Reference" "D106" (at 153.67 90.17 0)
       (effects (font (size 1.27 1.27)))
@@
   )
   (symbol (lib_id "LED:SK6812MINI") (at 151.13 58.42 0) (unit 1)
-    (in_bom yes) (on_board yes) (dnp no)
+    (in_bom no) (on_board yes) (dnp no)
     (property "Reference" "D105" (at 158.75 62.23 0)
       (effects (font (size 1.27 1.27)))

Commit message: update 3d models
Parts:
- D101, D102, D103, D104, D105, D106, D107, D108, D109, D110, D111: footprint LED_SMD:LED_SK6812MINI_PLCC4_3.5x3.5mm_P1.75mm -> modified_footrprints:LED_SK6812MINI_PLCC4_3.5x3.5mm_P1.75mm
Changed lines of the file:
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@@
       (effects (font (size 0.8 0.8)))
     )
-    (property "Footprint" "LED_SMD:LED_SK6812MINI_PLCC4_3.5x3.5mm_P1.75mm" (at 99.06 66.04 0)
+    (property "Footprint" "modified_footrprints:LED_SK6812MINI_PLCC4_3.5x3.5mm_P1.75mm" (at 99.06 66.04 0)
       (effects (font (size 1.27 1.27)) (justify left top) hide)
     )
@@
       (effects (font (size 0.8 0.8)) hide)
     )
-    (property "Footprint" "LED_SMD:LED_SK6812MINI_PLCC4_3.5x3.5mm_P1.75mm" (at 88.9 93.98 0)
+    (property "Footprint" "modified_footrprints:LED_SK6812MINI_PLCC4_3.5x3.5mm_P1.75mm" (at 88.9 93.98 0)
       (effects (font (size 1.27 1.27)) (justify left top) hide)
     )
@@
       (effects (font (size 0.8 0.8)) hide)
     )
-    (property "Footprint" "LED_SMD:LED_SK6812MINI_PLCC4_3.5x3.5mm_P1.75mm" (at 71.12 93.98 0)
+    (property "Footprint" "modified_footrprints:LED_SK6812MINI_PLCC4_3.5x3.5mm_P1.75mm" (at 71.12 93.98 0)
       (effects (font (size 1.27 1.27)) (justify left top) hide)
     )
@@
       (effects (font (size 0.8 0.8)))
     )
-    (property "Footprint" "LED_SMD:LED_SK6812MINI_PLCC4_3.5x3.5mm_P1.75mm" (at 106.68 93.98 0)
+    (property "Footprint" "modified_footrprints:LED_SK6812MINI_PLCC4_3.5x3.5mm_P1.75mm" (at 106.68 93.98 0)
       (effects (font (size 1.27 1.27)) (justify left top) hide)
     )
@@
       (effects (font (size 0.8 0.8)))
     )
-    (property "Footprint" "LED_SMD:LED_SK6812MINI_PLCC4_3.5x3.5mm_P1.75mm" (at 116.84 66.04 0)
+    (property "Footprint" "modified_footrprints:LED_SK6812MINI_PLCC4_3.5x3.5mm_P1.75mm" (at 116.84 66.04 0)
       (effects (font (size 1.27 1.27)) (justify left top) hide)
     )
@@
       (effects (font (size 0.8 0.8)))
     )
-    (property "Footprint" "LED_SMD:LED_SK6812MINI_PLCC4_3.5x3.5mm_P1.75mm" (at 142.24 93.98 0)
+    (property "Footprint" "modified_footrprints:LED_SK6812MINI_PLCC4_3.5x3.5mm_P1.75mm" (at 142.24 93.98 0)
       (effects (font (size 1.27 1.27)) (justify left top) hide)
     )
@@
       (effects (font (size 0.8 0.8)))
     )
-    (property "Footprint" "LED_SMD:LED_SK6812MINI_PLCC4_3.5x3.5mm_P1.75mm" (at 134.62 66.04 0)
+    (property "Footprint" "modified_footrprints:LED_SK6812MINI_PLCC4_3.5x3.5mm_P1.75mm" (at 134.62 66.04 0)
       (effects (font (size 1.27 1.27)) (justify left top) hide)
     )
@@
       (effects (font (size 0.8 0.8)))
     )
-    (property "Footprint" "LED_SMD:LED_SK6812MINI_PLCC4_3.5x3.5mm_P1.75mm" (at 124.46 93.98 0)
+    (property "Footprint" "modified_footrprints:LED_SK6812MINI_PLCC4_3.5x3.5mm_P1.75mm" (at 124.46 93.98 0)
       (effects (font (size 1.27 1.27)) (justify left top) hide)
     )
@@
       (effects (font (size 0.8 0.8)))
     )
-    (property "Footprint" "LED_SMD:LED_SK6812MINI_PLCC4_3.5x3.5mm_P1.75mm" (at 81.28 66.04 0)
+    (property "Footprint" "modified_footrprints:LED_SK6812MINI_PLCC4_3.5x3.5mm_P1.75mm" (at 81.28 66.04 0)
       (effects (font (size 1.27 1.27)) (justify left top) hide)
     )
@@
       (effects (font (size 0.8 0.8)))
     )
-    (property "Footprint" "LED_SMD:LED_SK6812MINI_PLCC4_3.5x3.5mm_P1.75mm" (at 160.02 93.98 0)
+    (property "Footprint" "modified_footrprints:LED_SK6812MINI_PLCC4_3.5x3.5mm_P1.75mm" (at 160.02 93.98 0)
       (effects (font (size 1.27 1.27)) (justify left top) hide)
     )
@@
       (effects (font (size 0.8 0.8)))
     )
-    (property "Footprint" "LED_SMD:LED_SK6812MINI_PLCC4_3.5x3.5mm_P1.75mm" (at 152.4 66.04 0)
-      (effects (font (size 1.27 1.27)) (justify left top) hide)
-    )
+    (property "Footprint" "modified_footrprints:LED_SK6812MINI_PLCC4_3.5x3.5mm_P1.75mm" (at 152.4 66.04 0)
+      (effects (font (size 1.27 1.27)) (justify left top) hide)
+    )

Commit message: v0.2
Parts:
- D101, D102: now in the parts list
- D103, D105, D106: JlcRotOffset (none) -> -14; now in the parts list
- D104: JlcRotOffset (none) -> 166; now in the parts list
- D107: JlcRotOffset (none) -> 180; now in the parts list
- D108, D109, D111: JlcRotOffset (none) -> 14; now in the parts list
- D110: JlcRotOffset (none) -> 194; now in the parts list
Other:
- company: (none) -> sporkus
- title: (none) -> Hotswap Chiffre

Commit message: adding front LED bypass jumper
Parts:
- added JP2: Jumper_2_Open, Jumper:SolderJumper-2_P1.3mm_Open_TrianglePad1.0x1.5mm, symbol Jumper:Jumper_2_Open
Connections:
- net RGB: now also JP2.1 (A)
- net at D102.1 (DOUT), D103.3 (DIN): now also JP2.2 (B)
Changed lines of the file:
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@@
   (title_block
     (title "Hotswap Chiffre")
-    (date "2023-07-07")
-    (rev "0.2")
+    (date "2023-07-13")
+    (rev "0.2.1")
     (company "sporkus")
   )
@@
   (junction (at 125.73 78.74) (diameter 0) (color 0 0 0 0)
   )
+  (junction (at 66.929 40.132) (diameter 0) (color 0 0 0 0)
+  )
   (junction (at 80.01 50.8) (diameter 0) (color 0 0 0 0)
   )
@@
   (junction (at 80.01 66.04) (diameter 0) (color 0 0 0 0)
   )
+  (junction (at 107.188 58.42) (diameter 0) (color 0 0 0 0)
+  )
   (junction (at 143.51 93.98) (diameter 0) (color 0 0 0 0)
   )
@@
     (stroke (width 0) (type default))
   )
+  (wire (pts (xy 66.929 40.132) (xy 97.028 40.132))
+    (stroke (width 0) (type default))
+  )
   (wire (pts (xy 125.73 93.98) (xy 143.51 93.98))
     (stroke (width 0) (type default))
@@
     (stroke (width 0) (type default))
   )
+  (wire (pts (xy 107.188 58.42) (xy 107.95 58.42))
+    (stroke (width 0) (type default))
+  )
   (wire (pts (xy 140.97 58.42) (xy 143.51 58.42))
     (stroke (width 0) (type default))
   )
+  (wire (pts (xy 66.929 58.42) (xy 72.39 58.42))
+    (stroke (width 0) (type default))
+  )
   (wire (pts (xy 97.79 66.04) (xy 115.57 66.04))
     (stroke (width 0) (type default))
@@
     (stroke (width 0) (type default))
   )
+  (wire (pts (xy 66.929 40.132) (xy 66.929 58.42))
+    (stroke (width 0) (type default))
+  )
   (wire (pts (xy 80.01 48.26) (xy 80.01 50.8))
     (stroke (width 0) (type default))
@@
     (stroke (width 0) (type default))
   )
-  (wire (pts (xy 105.41 58.42) (xy 107.95 58.42))
+  (wire (pts (xy 105.41 58.42) (xy 107.188 58.42))
     (stroke (width 0) (type default))
   )
@@
     (stroke (width 0) (type default))
   )
-  (wire (pts (xy 71.12 58.42) (xy 72.39 58.42))
+  (wire (pts (xy 61.595 40.132) (xy 66.929 40.132))
     (stroke (width 0) (type default))
   )
@@
     (stroke (width 0) (type default))
   )
+  (wire (pts (xy 107.188 40.132) (xy 107.188 58.42))
+    (stroke (width 0) (type default))
+  )
   (wire (pts (xy 90.17 78.74) (xy 107.95 78.74))
     (stroke (width 0) (type default))
@@
     (stroke (width 0) (type default))
   )
-  (global_label "RGB" (shape input) (at 71.12 58.42 180)
+  (global_label "RGB" (shape input) (at 61.595 40.132 180)
     (effects (font (size 1.27 1.27)) (justify right))
-    (property "Intersheetrefs" "${INTERSHEET_REFS}" (at 71.12 58.42 0)
+    (property "Intersheetrefs" "${INTERSHEET_REFS}" (at 61.595 40.132 0)
       (effects (font (size 1.27 1.27)) hide)
     )
@@
         )
       )
+    )
+  )
+  (symbol (lib_id "Jumper:Jumper_2_Open") (at 102.108 40.132 0) (unit 1)
+    (in_bom yes) (on_board yes) (dnp no) (fields_autoplaced)
+    (property "Reference" "JP2" (at 102.108 34.163 0)
+      (effects (font (size 1.27 1.27)))
+    )
+    (property "Value" "Jumper_2_Open" (at 102.108 36.703 0)
+      (effects (font (size 1.27 1.27)))
+    )
+    (property "Footprint" "Jumper:SolderJumper-2_P1.3mm_Open_TrianglePad1.0x1.5mm" (at 102.108 40.132 0)
+      (effects (font (size 1.27 1.27)) hide)
+    )
+    (property "Datasheet" "~" (at 102.108 40.132 0)
+      (effects (font (size 1.27 1.27)) hide)
+    )
+    (pin "1")
+    (pin "2")
+    (instances
+      (project "stm32_hotswap_chiffre"
+        (path "/ca0d59d2-7f9b-4344-99bc-39bc2c8c88cb/ec6e930e-09f1-49e7-aa49-9ca6fe61b6ec"
+          (reference "JP2") (unit 1)
+        )
+      )
