File: kicad/pcb/stm32_hotswap_chiffre.kicad_pcb (KiCad board)
At the start: 2 copper layers, 227.4 x 84.9 mm, 109 parts, among them J1 USB_C_Receptacle_USB2.0, J101 Conn_01x03_Female, J2 OLED I2C, SW1 SW_Push, SW10 SW_Push, SW11 SW_Push, SW12 SW_Push, SW13 SW_Push, SW14 SW_Push, SW15 SW_Push, SW16 SW_Push, SW17 SW_Push, SW18 SW_Push, SW19 SW_Push, SW2 SW_Push, SW20 SW_Push, SW21 SW_Push, SW22 SW_Push, SW23 SW_Push, SW24 SW_Push, SW25 SW_Push, SW26 SW_Push, SW27 SW_Push, SW28 SW_Push, SW29 SW_Push, SW3 SW_Push, SW30 SW_Push, SW31 SW_Push, SW32 SW_Push, SW33 SW_Push, SW34 SW_Push, SW35 SW_Push, SW36 Rotary_Encoder_Switch, SW37 SKQGABE010, SW4 SW_Push, SW5 SW_Push, SW6 SW_Push, SW7 SW_Push, SW8 SW_Push, SW9 SW_Push, U1 STM32F072CBT6, U2 PRTR5V0U2X, U3 XC6206PxxxMR-Regulator_Linear

Commit message: add QR code
Parts:
- added G***: LOGO, LOGO, B.Cu at (162.6, 135.9)

Commit message: Initial SAM/nRF52 version.
Parts:
- removed the C7 at (153.2, 124.2)
- removed the C9 at (151.2, 92.4)
- removed D101, D102, D103, D104, D105, D106, D107, D108, D109, D110, D111: SK6812MINI, modified_footrprints:LED_SK6812MINI_PLCC4_3.5x3.5mm_P1.75mm
- removed G***: LOGO, LOGO
- removed J101: Conn_01x03_Female, Connector_PinSocket_2.54mm:PinSocket_1x03_P2.54mm_Vertical
- removed SW36: Rotary_Encoder_Switch, modified_footprints:RotaryEncoder_EC11_no_mp
- removed U1: STM32F072CBT6, Package_QFP:LQFP-48_7x7mm_P0.5mm
- added C11: 4.7uF, Capacitor_SMD:C_0805_2012Metric, F.Cu at (132.6, 105.7)
- added C12: 12pF, Capacitor_SMD:C_0805_2012Metric, F.Cu at (132.1, 116.4)
- added C13: 12pF, Capacitor_SMD:C_0805_2012Metric, F.Cu at (132.1, 118.3)
- added D36: Charge, LED_SMD:LED_0805_2012Metric, F.Cu at (146.6, 101.2)
- added D37: BAT54HT1G, Diode_SMD:D_SOD-323, F.Cu at (135.7, 102.8)
- added D38: User, LED_SMD:LED_0805_2012Metric, F.Cu at (146.6, 103.3)
- added J3: nRF52, PCM_marbastlib-various:CON_TC2030_outlined, F.Cu at (161.7, 116.5)
- added J4: Conn_01x02_Socket, Connector_JST:JST_SH_BM02B-SRSS-TB_1x02-1MP_P1.00mm_Vertical, F.Cu at (125.4, 142.8)
- added J5: Conn_01x02_Socket, Connector_PinHeader_2.54mm:PinHeader_1x02_P2.54mm_Vertical, F.Cu at (126.1, 135.5)
- added JP3: Wired, Jumper:SolderJumper-2_P1.3mm_Open_TrianglePad1.0x1.5mm, B.Cu at (155.0, 98.9)
- added JP4: Wireless, Jumper:SolderJumper-2_P1.3mm_Open_TrianglePad1.0x1.5mm, B.Cu at (157.6, 98.9)
- added L2: 10uH, Inductor_SMD:L_0805_2012Metric, B.Cu at (155.6, 112.4)
- added Q2: AO3401A, Package_TO_SOT_SMD:SOT-23, F.Cu at (135.6, 105.7)
- added R10: R_Small, Resistor_SMD:R_0805_2012Metric, F.Cu at (143.1, 103.2)
- added R11: 1k, Resistor_SMD:R_0805_2012Metric, B.Cu at (163.2, 111.7)
- added R6: 806k, Resistor_SMD:R_0805_2012Metric, F.Cu at (134.7, 109.2)
- added R7: 2M, Resistor_SMD:R_0805_2012Metric, F.Cu at (136.7, 109.2)
- added R8: 4.7k, Resistor_SMD:R_0805_2012Metric, B.Cu at (143.6, 106.3)
- added R9: 9k, Resistor_SMD:R_0805_2012Metric, B.Cu at (145.6, 106.3)
- added U4: ATSAML21E18B-AUT, Package_QFP:TQFP-32_7x7mm_P0.8mm, B.Cu at (146.6, 113.3)
- added U5: BC805M, Fanstel_modules:BC805M, F.Cu at (151.6, 111.9)
- added U6: MCP73832-2-OT, Package_TO_SOT_SMD:SOT-23-5, F.Cu at (135.8, 99.7)
- added U7: 74LVC1G08, Package_TO_SOT_SMD:SOT-23-5_HandSoldering, B.Cu at (129.6, 107.0)
- added U8: 74LVC1G08, Package_TO_SOT_SMD:SOT-23-5_HandSoldering, B.Cu at (133.2, 107.0)
- added U9: 74LVC1G08, Package_TO_SOT_SMD:SOT-23-5_HandSoldering, B.Cu at (131.4, 111.9)
- added Y2: 32.768 kHz, Crystal:Crystal_SMD_2012-2Pin_2.0x1.2mm_HandSoldering, F.Cu at (134.8, 117.5)
- C1, C2, C8: footprint Capacitor_SMD:C_0402_1005Metric -> Capacitor_SMD:C_0805_2012Metric
- C10: value 100nF -> 4.7uF; footprint Capacitor_SMD:C_0402_1005Metric -> Capacitor_SMD:C_0805_2012Metric; moved to F.Cu
- C3, C4: value 100nF -> 10uF; footprint Capacitor_SMD:C_0402_1005Metric -> Capacitor_SMD:C_0805_2012Metric
- C5: value 100nF -> 1uF; footprint Capacitor_SMD:C_0402_1005Metric -> Capacitor_SMD:C_0805_2012Metric
- C6: footprint Capacitor_SMD:C_0603_1608Metric -> Capacitor_SMD:C_0805_2012Metric; moved to F.Cu
- C7: renamed from C11; footprint Capacitor_SMD:C_0402_1005Metric -> Capacitor_SMD:C_0805_2012Metric
- C9: renamed from C12; footprint Capacitor_SMD:C_0402_1005Metric -> Capacitor_SMD:C_0805_2012Metric
- J2: value OLED I2C -> SAM; footprint Connector_PinHeader_2.54mm:PinHeader_1x04_P2.54mm_Vertical -> PCM_marbastlib-various:CON_TC2030_outlined
- JP2: value Jumper_2_Open -> Wired; moved to B.Cu
- R1, R2: footprint Resistor_SMD:R_0402_1005Metric -> Resistor_SMD:R_0805_2012Metric
- R3: value 10k -> R_Small; footprint Resistor_SMD:R_0402_1005Metric -> Resistor_SMD:R_0805_2012Metric; moved to F.Cu
- R4: value 4.7k -> 10k; footprint Resistor_SMD:R_0402_1005Metric -> Resistor_SMD:R_0805_2012Metric; moved to F.Cu
- R5: value 4.7k -> 100k; footprint Resistor_SMD:R_0402_1005Metric -> Resistor_SMD:R_0805_2012Metric; moved to F.Cu
- SW33: renamed from SW35; footprint MX_Alps_Hybrid:MX-Alps-Hybrid-1U -> MX_hotswap_alps:MX-Hotswap-Alps-1U
- SW37: value SKQGABE010 -> Reset
- moved C7 32.7 mm to (159.6, 105.5), turned to 90 degrees
- moved U3 31.1 mm to (156.5, 105.5), turned to 0 degrees
- moved C9 29.3 mm to (153.4, 105.5)
- moved J2 27.7 mm to (161.7, 116.5), turned to 0 degrees
- moved C4 17.3 mm to (137.8, 115.0)
- moved C1 15.9 mm to (153.4, 116.1), turned to -90 degrees
- moved R5 15.3 mm to (138.7, 105.7)
- moved JP2 13.6 mm to (158.1, 112.4), turned to -90 degrees
- moved R4 12.5 mm to (139.0, 99.7), turned to 90 degrees
- moved C10 12.1 mm to (132.3, 99.7), turned to 90 degrees
- moved C6 11.6 mm to (139.8, 113.1)
- moved D33 11.2 mm to (140.6, 88.7), turned to 90 degrees
- moved R3 8.58 mm to (143.1, 101.2), turned to 0 degrees
- moved C5 7.20 mm to (153.5, 112.4)
- moved C3 6.69 mm to (155.6, 116.1), turned to -90 degrees
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- renumbered D35 to D33, D33 to D34, D34 to D35, SW33 to SW34, SW34 to SW35
Connections:
- C1 pad 2: GND -> -BATT
- C10 pad 1: EncA -> +BATT
- C10 pad 2: GND -> -BATT
- C2 pad 2: GND -> -BATT
- C3 pad 2: GND -> -BATT
- C4 pad 2: GND -> -BATT
- C5 pad 1: +3V3 -> -BATT
- C5 pad 2: GND -> Net-(JP2-A)
- C6 pad 1: +3V3 -> -BATT
- C6 pad 2: GND -> +3V3
- C7 pad 1: GND -> -BATT
- C7 pad 2: +5V -> Net-(JP3-B)
- C8 pad 2: GND -> -BATT
- C9 pad 1: GND -> -BATT
- D1 pad 1: Net-(D1-K) -> row0_l
- D1 pad 2: row0 -> Net-(D1-A)
- D10 pad 1: Net-(D10-K) -> row0_r
- D10 pad 2: row0 -> Net-(D10-A)
- D11 pad 1: Net-(D11-K) -> row1_l
- D11 pad 2: row1 -> Net-(D11-A)
- D12 pad 1: Net-(D12-K) -> row1_l
- D12 pad 2: row1 -> Net-(D12-A)
- D13 pad 1: Net-(D13-K) -> row1_l
- D13 pad 2: row1 -> Net-(D13-A)
- D14 pad 1: Net-(D14-K) -> row1_l
- D14 pad 2: row1 -> Net-(D14-A)
- D15 pad 1: Net-(D15-K) -> row1_l
- D15 pad 2: row1 -> Net-(D15-A)
- D16 pad 1: Net-(D16-K) -> row1_r
- D16 pad 2: row1 -> Net-(D16-A)
- D17 pad 1: Net-(D17-K) -> row1_r
- D17 pad 2: row1 -> Net-(D17-A)
- D18 pad 1: Net-(D18-K) -> row1_r
- D18 pad 2: row1 -> Net-(D18-A)
- D19 pad 1: Net-(D19-K) -> row1_r
- D19 pad 2: row1 -> Net-(D19-A)
- D2 pad 1: Net-(D2-K) -> row0_l
- D2 pad 2: row0 -> Net-(D2-A)
- D20 pad 1: Net-(D20-K) -> row1_r
- D20 pad 2: row1 -> Net-(D20-A)
- D21 pad 1: Net-(D21-K) -> row2_l
- D21 pad 2: row2 -> Net-(D21-A)
- D22 pad 1: Net-(D22-K) -> row2_l
- D22 pad 2: row2 -> Net-(D22-A)
- D23 pad 1: Net-(D23-K) -> row2_l
- D23 pad 2: row2 -> Net-(D23-A)
- D24 pad 1: Net-(D24-K) -> row2_l
- D24 pad 2: row2 -> Net-(D24-A)
- D25 pad 1: Net-(D25-K) -> row2_l
- D25 pad 2: row2 -> Net-(D25-A)
- D26 pad 1: Net-(D26-K) -> row2_r
- D26 pad 2: row2 -> Net-(D26-A)
- D27 pad 1: Net-(D27-K) -> row2_r
- D27 pad 2: row2 -> Net-(D27-A)
- D28 pad 1: Net-(D28-K) -> row2_r
- D28 pad 2: row2 -> Net-(D28-A)
- D29 pad 1: Net-(D29-K) -> row2_r
- D29 pad 2: row2 -> Net-(D29-A)
- D3 pad 1: Net-(D3-K) -> row0_l
- D3 pad 2: row0 -> Net-(D3-A)
- D30 pad 1: Net-(D30-K) -> row2_r
- D30 pad 2: row2 -> Net-(D30-A)
- D31 pad 1: Net-(D31-K) -> row3
- D31 pad 2: row3 -> Net-(D31-A)
- D32 pad 1: Net-(D32-K) -> row3
- D32 pad 2: row3 -> Net-(D32-A)
- D33 pad 1: Net-(D35-K) -> row3
- D33 pad 2: row3 -> Net-(D33-A)
- D34 pad 1: Net-(D33-K) -> row3
- D34 pad 2: row3 -> Net-(D34-A)
- D35 pad 1: Net-(D34-K) -> row3
- D35 pad 2: row3 -> Net-(D35-A)
- D4 pad 1: Net-(D4-K) -> row0_l
- D4 pad 2: row0 -> Net-(D4-A)
- D5 pad 1: Net-(D5-K) -> row0_l
- D5 pad 2: row0 -> Net-(D5-A)
- D6 pad 1: Net-(D6-K) -> row0_r
- D6 pad 2: row0 -> Net-(D6-A)
- D7 pad 1: Net-(D7-K) -> row0_r
- D7 pad 2: row0 -> Net-(D7-A)
- D8 pad 1: Net-(D8-K) -> row0_r
- D8 pad 2: row0 -> Net-(D8-A)
- D9 pad 1: Net-(D9-K) -> row0_r
- D9 pad 2: row0 -> Net-(D9-A)
- J1 pad A1: GND -> GNDPWR
- J1 pad A12: GND -> GNDPWR
- J1 pad B1: GND -> GNDPWR
- J1 pad B12: GND -> GNDPWR
- J1 pad S1: GND -> GNDPWR
- J2 pad 1: GND -> +3V3
- J2 pad 2: +3V3 -> /SWDIO
- J2 pad 3: SCL -> /RESET
- J2 pad 4: SDA -> /SWCLK
- JP2 pad 1: RGB -> Net-(JP2-A)
- L1 pad 1: GND -> GNDPWR
- L1 pad 2: GND -> -BATT
- R1 pad 1: GND -> -BATT
- R2 pad 1: GND -> -BATT
- R3 pad 1: BOOT0 -> +5V
- R3 pad 2: GND -> Net-(D36-A)
- R4 pad 1: SDA -> Net-(U6-PROG)
- R4 pad 2: +3V3 -> -BATT
- R5 pad 1: SCL -> +5V
- R5 pad 2: +3V3 -> -BATT
- SW1 pad 1: Net-(D1-K) -> Net-(D1-A)
- SW10 pad 1: Net-(D10-K) -> Net-(D10-A)
- SW10 pad 2: col9 -> col0
- SW11 pad 1: Net-(D11-K) -> Net-(D11-A)
- SW12 pad 1: Net-(D12-K) -> Net-(D12-A)
- SW13 pad 1: Net-(D13-K) -> Net-(D13-A)
- SW14 pad 1: Net-(D14-K) -> Net-(D14-A)
- SW15 pad 1: Net-(D15-K) -> Net-(D15-A)
- SW16 pad 1: Net-(D16-K) -> Net-(D16-A)
- SW16 pad 2: col5 -> col4
- SW17 pad 1: Net-(D17-K) -> Net-(D17-A)
- SW17 pad 2: col6 -> col3
- SW18 pad 1: Net-(D18-K) -> Net-(D18-A)
- SW18 pad 2: col7 -> col2
- SW19 pad 1: Net-(D19-K) -> Net-(D19-A)
- SW19 pad 2: col8 -> col1
- SW2 pad 1: Net-(D2-K) -> Net-(D2-A)
- SW20 pad 1: Net-(D20-K) -> Net-(D20-A)
- SW20 pad 2: col9 -> col0
- SW21 pad 1: Net-(D21-K) -> Net-(D21-A)
- SW22 pad 1: Net-(D22-K) -> Net-(D22-A)
- SW23 pad 1: Net-(D23-K) -> Net-(D23-A)
- SW24 pad 1: Net-(D24-K) -> Net-(D24-A)
- SW25 pad 1: Net-(D25-K) -> Net-(D25-A)
- SW26 pad 1: Net-(D26-K) -> Net-(D26-A)
- SW26 pad 2: col5 -> col4
- SW27 pad 1: Net-(D27-K) -> Net-(D27-A)
- SW27 pad 2: col6 -> col3
- SW28 pad 1: Net-(D28-K) -> Net-(D28-A)
- SW28 pad 2: col7 -> col2
- SW29 pad 1: Net-(D29-K) -> Net-(D29-A)
- SW29 pad 2: col8 -> col1
- SW3 pad 1: Net-(D3-K) -> Net-(D3-A)
- SW30 pad 1: Net-(D30-K) -> Net-(D30-A)
- SW30 pad 2: col9 -> col0
- SW31 pad 1: Net-(D31-K) -> Net-(D31-A)
- SW31 pad 2: col2 -> col0
- SW32 pad 1: Net-(D32-K) -> Net-(D32-A)
- SW32 pad 2: col4 -> col1
- SW33 pad 1: Net-(D35-K) -> Net-(D33-A)
- SW33 pad 2: col5 -> col2
- SW34 pad 1: Net-(D33-K) -> Net-(D34-A)
- SW34 pad 2: col6 -> col4
- SW35 pad 1: Net-(D34-K) -> Net-(D35-A)
- SW35 pad 2: col7 -> col3
- SW37 pad 1: +3V3 -> /RESET
- SW37 pad 2: BOOT0 -> -BATT
- SW4 pad 1: Net-(D4-K) -> Net-(D4-A)
- SW5 pad 1: Net-(D5-K) -> Net-(D5-A)
- SW6 pad 1: Net-(D6-K) -> Net-(D6-A)
- SW6 pad 2: col5 -> col4
- SW7 pad 1: Net-(D7-K) -> Net-(D7-A)
- SW7 pad 2: col6 -> col3
- SW8 pad 1: Net-(D8-K) -> Net-(D8-A)
- SW8 pad 2: col7 -> col2
- SW9 pad 1: Net-(D9-K) -> Net-(D9-A)
- SW9 pad 2: col8 -> col1
- U3 pad 1: GND -> -BATT
- U3 pad 3: +5V -> Net-(JP3-B)
Routing:
- net +5V: track 649.1 -> 75.5 mm, vias 16 -> 2
- net row0: track 294.9 -> 0.00 mm, vias 6 -> 0
- net row1: track 276.3 -> 0.00 mm, vias 6 -> 0
- net col0: track 160.5 -> 425.5 mm, vias 0 -> 1
- net col1: track 138.7 -> 374.0 mm, vias 1 -> 3
- net row2: track 230.3 -> 0.00 mm, vias 4 -> 0
- net Net-(D30-A): track 0.00 -> 167.7 mm, vias 0 -> 2
- net col9: track 163.1 -> 0.00 mm
- net col7: track 160.3 -> 0.00 mm
- net col3: track 99.5 -> 258.4 mm, vias 0 -> 1
- net Net-(D10-A): track 0.00 -> 142.6 mm, vias 0 -> 2
- net col8: track 140.9 -> 0.00 mm, vias 1 -> 0
- net col5: track 140.6 -> 0.00 mm, vias 5 -> 0
- net col2: track 138.3 -> 277.8 mm, vias 0 -> 2
- net col6: track 137.7 -> 0.00 mm, vias 1 -> 0
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- added copper zone on B.Cu, net -BATT
- added copper zone on F.Cu, net -BATT
- removed copper zone on B.Cu, net GND
- removed copper zone on F.Cu, net GND
Other:
- outline, holes or cut-outs redrawn
- board text added: "+ Red"
- board text added: "- Black"
- board text added: "Black -"
- board text added: "Red +"
- board text removed: "3v3"
- board text removed: "5v"
- board text removed: "DFU"
- board text removed: "JLCJLCJLCJLC"
- board text removed: "Le Chiffre 32 v0.2.2 by sporkus"
- board text removed: "front leds bypass"
- board text removed: "gnd"
- board text removed: "rgb_out"
- board text removed: "scl"
- board text removed: "sda"
