File: kicad/stm32_chiffre_36keys/rgb.kicad_sch (KiCad schematic)
At the start: 13 parts, among them J101 Conn_01x03_Female

Commit message: fix schematic on right thumb keys
Other:
- title: Hotswap Chiffre -> Hotswap Chiffre (36 key)
Changed lines of the file:
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@@
   (paper "A4")
   (title_block
-    (title "Hotswap Chiffre")
-    (date "2023-07-13")
-    (rev "0.2.2")
+    (title "Hotswap Chiffre (36 key)")
+    (date "2024-03-06")
+    (rev "0.3")
     (company "sporkus")
   )
@@
     (pin "1")
     (instances
-      (project "stm32_hotswap_chiffre"
+      (project "stm32_chiffre_36keys"
         (path "/ca0d59d2-7f9b-4344-99bc-39bc2c8c88cb/ec6e930e-09f1-49e7-aa49-9ca6fe61b6ec"
           (reference "#PWR0101") (unit 1)
@@
     (pin "4")
     (instances
-      (project "stm32_hotswap_chiffre"
+      (project "stm32_chiffre_36keys"
         (path "/ca0d59d2-7f9b-4344-99bc-39bc2c8c88cb/ec6e930e-09f1-49e7-aa49-9ca6fe61b6ec"
           (reference "D104") (unit 1)
@@
     (pin "4")
     (instances
-      (project "stm32_hotswap_chiffre"
+      (project "stm32_chiffre_36keys"
         (path "/ca0d59d2-7f9b-4344-99bc-39bc2c8c88cb/ec6e930e-09f1-49e7-aa49-9ca6fe61b6ec"
           (reference "D102") (unit 1)
@@
     (pin "4")
     (instances
-      (project "stm32_hotswap_chiffre"
+      (project "stm32_chiffre_36keys"
         (path "/ca0d59d2-7f9b-4344-99bc-39bc2c8c88cb/ec6e930e-09f1-49e7-aa49-9ca6fe61b6ec"
           (reference "D103") (unit 1)
@@
     (pin "3")
     (instances
-      (project "stm32_hotswap_chiffre"
+      (project "stm32_chiffre_36keys"
         (path "/ca0d59d2-7f9b-4344-99bc-39bc2c8c88cb/ec6e930e-09f1-49e7-aa49-9ca6fe61b6ec"
           (reference "J101") (unit 1)
@@
     (pin "4")
     (instances
-      (project "stm32_hotswap_chiffre"
+      (project "stm32_chiffre_36keys"
         (path "/ca0d59d2-7f9b-4344-99bc-39bc2c8c88cb/ec6e930e-09f1-49e7-aa49-9ca6fe61b6ec"
           (reference "D108") (unit 1)
@@
     (pin "4")
     (instances
-      (project "stm32_hotswap_chiffre"
+      (project "stm32_chiffre_36keys"
         (path "/ca0d59d2-7f9b-4344-99bc-39bc2c8c88cb/ec6e930e-09f1-49e7-aa49-9ca6fe61b6ec"
           (reference "D106") (unit 1)
@@
     (pin "4")
     (instances
-      (project "stm32_hotswap_chiffre"
+      (project "stm32_chiffre_36keys"
         (path "/ca0d59d2-7f9b-4344-99bc-39bc2c8c88cb/ec6e930e-09f1-49e7-aa49-9ca6fe61b6ec"
           (reference "D105") (unit 1)
@@
     (pin "1")
     (instances
-      (project "stm32_hotswap_chiffre"
+      (project "stm32_chiffre_36keys"
         (path "/ca0d59d2-7f9b-4344-99bc-39bc2c8c88cb/ec6e930e-09f1-49e7-aa49-9ca6fe61b6ec"
           (reference "#PWR0106") (unit 1)
@@
     (pin "1")
     (instances
-      (project "stm32_hotswap_chiffre"
+      (project "stm32_chiffre_36keys"
         (path "/ca0d59d2-7f9b-4344-99bc-39bc2c8c88cb/ec6e930e-09f1-49e7-aa49-9ca6fe61b6ec"
           (reference "#PWR019") (unit 1)
@@
     (pin "4")
     (instances
-      (project "stm32_hotswap_chiffre"
+      (project "stm32_chiffre_36keys"
         (path "/ca0d59d2-7f9b-4344-99bc-39bc2c8c88cb/ec6e930e-09f1-49e7-aa49-9ca6fe61b6ec"
           (reference "D107") (unit 1)
@@
     (pin "4")
     (instances
-      (project "stm32_hotswap_chiffre"
+      (project "stm32_chiffre_36keys"
         (path "/ca0d59d2-7f9b-4344-99bc-39bc2c8c88cb/ec6e930e-09f1-49e7-aa49-9ca6fe61b6ec"
           (reference "D110") (unit 1)
@@
     (pin "2")
     (instances
-      (project "stm32_hotswap_chiffre"
+      (project "stm32_chiffre_36keys"
         (path "/ca0d59d2-7f9b-4344-99bc-39bc2c8c88cb/ec6e930e-09f1-49e7-aa49-9ca6fe61b6ec"
           (reference "JP2") (unit 1)
@@
     (pin "4")
     (instances
-      (project "stm32_hotswap_chiffre"
+      (project "stm32_chiffre_36keys"
         (path "/ca0d59d2-7f9b-4344-99bc-39bc2c8c88cb/ec6e930e-09f1-49e7-aa49-9ca6fe61b6ec"
           (reference "D101") (unit 1)
@@
     (pin "4")
     (instances
-      (project "stm32_hotswap_chiffre"
+      (project "stm32_chiffre_36keys"
         (path "/ca0d59d2-7f9b-4344-99bc-39bc2c8c88cb/ec6e930e-09f1-49e7-aa49-9ca6fe61b6ec"
           (reference "D109") (unit 1)
@@
     (pin "4")
     (instances
-      (project "stm32_hotswap_chiffre"
+      (project "stm32_chiffre_36keys"
         (path "/ca0d59d2-7f9b-4344-99bc-39bc2c8c88cb/ec6e930e-09f1-49e7-aa49-9ca6fe61b6ec"
           (reference "D111") (unit 1)
@@
     (pin "1")
     (instances
-      (project "stm32_hotswap_chiffre"
+      (project "stm32_chiffre_36keys"
         (path "/ca0d59d2-7f9b-4344-99bc-39bc2c8c88cb/ec6e930e-09f1-49e7-aa49-9ca6fe61b6ec"
           (reference "#PWR0105") (unit 1)
@@
     (pin "1")
     (instances
-      (project "stm32_hotswap_chiffre"
+      (project "stm32_chiffre_36keys"
         (path "/ca0d59d2-7f9b-4344-99bc-39bc2c8c88cb/ec6e930e-09f1-49e7-aa49-9ca6fe61b6ec"
           (reference "#PWR0104") (unit 1)
@@
     (pin "1")
     (instances
-      (project "stm32_hotswap_chiffre"
+      (project "stm32_chiffre_36keys"
         (path "/ca0d59d2-7f9b-4344-99bc-39bc2c8c88cb/ec6e930e-09f1-49e7-aa49-9ca6fe61b6ec"
           (reference "#PWR0102") (unit 1)
@@
     (pin "1")
     (instances
-      (project "stm32_hotswap_chiffre"
+      (project "stm32_chiffre_36keys"
         (path "/ca0d59d2-7f9b-4344-99bc-39bc2c8c88cb/ec6e930e-09f1-49e7-aa49-9ca6fe61b6ec"
           (reference "#PWR020") (unit 1)
