File: kicad/stm32_chiffre_36keys/stm32_chiffre_36keys.kicad_sch (KiCad schematic)
At the start: 23 parts, among them J1 USB_C_Receptacle_USB2.0, J2 OLED I2C, U1 STM32F072CBT6, U2 PRTR5V0U2X

Commit message: fix schematic on right thumb keys
Other:
- title: Hotswap Chiffre -> Hotswap Chiffre (36 key)
Changed lines of the file:
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@@
   (paper "A4")
   (title_block
-    (title "Hotswap Chiffre")
-    (date "2023-07-13")
-    (rev "0.2.2")
+    (title "Hotswap Chiffre (36 key)")
+    (date "2024-03-06")
+    (rev "0.3")
     (company "sporkus")
   )
@@
         )
       )
-      (project "stm32_hotswap_chiffre"
+      (project "stm32_chiffre_36keys"
         (path "/ca0d59d2-7f9b-4344-99bc-39bc2c8c88cb"
           (reference "C11") (unit 1)
@@
     (pin "2")
     (instances
-      (project "stm32_hotswap_chiffre"
+      (project "stm32_chiffre_36keys"
         (path "/ca0d59d2-7f9b-4344-99bc-39bc2c8c88cb"
           (reference "L1") (unit 1)
@@
         )
       )
-      (project "stm32_hotswap_chiffre"
+      (project "stm32_chiffre_36keys"
         (path "/ca0d59d2-7f9b-4344-99bc-39bc2c8c88cb"
           (reference "#PWR011") (unit 1)
@@
         )
       )
-      (project "stm32_hotswap_chiffre"
+      (project "stm32_chiffre_36keys"
         (path "/ca0d59d2-7f9b-4344-99bc-39bc2c8c88cb"
           (reference "C12") (unit 1)
@@
     (pin "S1")
     (instances
-      (project "stm32_hotswap_chiffre"
+      (project "stm32_chiffre_36keys"
         (path "/ca0d59d2-7f9b-4344-99bc-39bc2c8c88cb"
           (reference "J1") (unit 1)
@@
     (pin "1")
     (instances
-      (project "stm32_hotswap_chiffre"
+      (project "stm32_chiffre_36keys"
         (path "/ca0d59d2-7f9b-4344-99bc-39bc2c8c88cb"
           (reference "#PWR08") (unit 1)
@@
     (pin "4")
     (instances
-      (project "stm32_hotswap_chiffre"
+      (project "stm32_chiffre_36keys"
         (path "/ca0d59d2-7f9b-4344-99bc-39bc2c8c88cb"
           (reference "U2") (unit 1)
@@
     (pin "2")
     (instances
-      (project "stm32_hotswap_chiffre"
+      (project "stm32_chiffre_36keys"
         (path "/ca0d59d2-7f9b-4344-99bc-39bc2c8c88cb"
           (reference "R5") (unit 1)
@@
     (pin "9")
     (instances
-      (project "stm32_hotswap_chiffre"
+      (project "stm32_chiffre_36keys"
         (path "/ca0d59d2-7f9b-4344-99bc-39bc2c8c88cb"
           (reference "U1") (unit 1)
@@
     (pin "1")
     (instances
-      (project "stm32_hotswap_chiffre"
+      (project "stm32_chiffre_36keys"
         (path "/ca0d59d2-7f9b-4344-99bc-39bc2c8c88cb"
           (reference "#PWR016") (unit 1)
@@
     (pin "1")
     (instances
-      (project "stm32_hotswap_chiffre"
+      (project "stm32_chiffre_36keys"
         (path "/ca0d59d2-7f9b-4344-99bc-39bc2c8c88cb"
           (reference "#PWR014") (unit 1)
@@
     (pin "1")
     (instances
-      (project "stm32_hotswap_chiffre"
+      (project "stm32_chiffre_36keys"
         (path "/ca0d59d2-7f9b-4344-99bc-39bc2c8c88cb"
           (reference "#PWR018") (unit 1)
@@
         )
       )
-      (project "stm32_hotswap_chiffre"
+      (project "stm32_chiffre_36keys"
         (path "/ca0d59d2-7f9b-4344-99bc-39bc2c8c88cb"
           (reference "C4") (unit 1)
@@
         )
       )
-      (project "stm32_hotswap_chiffre"
+      (project "stm32_chiffre_36keys"
         (path "/ca0d59d2-7f9b-4344-99bc-39bc2c8c88cb"
           (reference "#PWR012") (unit 1)
@@
         )
       )
-      (project "stm32_hotswap_chiffre"
+      (project "stm32_chiffre_36keys"
         (path "/ca0d59d2-7f9b-4344-99bc-39bc2c8c88cb"
           (reference "U3") (unit 1)
@@
         )
       )
-      (project "stm32_hotswap_chiffre"
+      (project "stm32_chiffre_36keys"
         (path "/ca0d59d2-7f9b-4344-99bc-39bc2c8c88cb"
           (reference "#PWR05") (unit 1)
@@
     (pin "1")
     (instances
-      (project "stm32_hotswap_chiffre"
+      (project "stm32_chiffre_36keys"
         (path "/ca0d59d2-7f9b-4344-99bc-39bc2c8c88cb"
           (reference "#PWR03") (unit 1)
@@
     (pin "1")
     (instances
-      (project "stm32_hotswap_chiffre"
+      (project "stm32_chiffre_36keys"
         (path "/ca0d59d2-7f9b-4344-99bc-39bc2c8c88cb"
           (reference "#PWR04") (unit 1)
@@
     (pin "1")
     (instances
-      (project "stm32_hotswap_chiffre"
+      (project "stm32_chiffre_36keys"
         (path "/ca0d59d2-7f9b-4344-99bc-39bc2c8c88cb"
           (reference "#PWR01") (unit 1)
@@
         )
       )
-      (project "stm32_hotswap_chiffre"
+      (project "stm32_chiffre_36keys"
         (path "/ca0d59d2-7f9b-4344-99bc-39bc2c8c88cb"
           (reference "R2") (unit 1)
@@
     (pin "1")
     (instances
-      (project "stm32_hotswap_chiffre"
+      (project "stm32_chiffre_36keys"
         (path "/ca0d59d2-7f9b-4344-99bc-39bc2c8c88cb"
           (reference "#PWR015") (unit 1)
@@
     (pin "1")
     (instances
-      (project "stm32_hotswap_chiffre"
+      (project "stm32_chiffre_36keys"
         (path "/ca0d59d2-7f9b-4344-99bc-39bc2c8c88cb"
           (reference "#PWR09") (unit 1)
@@
         )
       )
-      (project "stm32_hotswap_chiffre"
+      (project "stm32_chiffre_36keys"
         (path "/ca0d59d2-7f9b-4344-99bc-39bc2c8c88cb"
           (reference "C3") (unit 1)
@@
     (pin "1")
     (instances
-      (project "stm32_hotswap_chiffre"
+      (project "stm32_chiffre_36keys"
         (path "/ca0d59d2-7f9b-4344-99bc-39bc2c8c88cb"
           (reference "#PWR021") (unit 1)
@@
         )
       )
-      (project "stm32_hotswap_chiffre"
+      (project "stm32_chiffre_36keys"
         (path "/ca0d59d2-7f9b-4344-99bc-39bc2c8c88cb"
           (reference "C1") (unit 1)
@@
     (pin "1")
     (instances
-      (project "stm32_hotswap_chiffre"
+      (project "stm32_chiffre_36keys"
         (path "/ca0d59d2-7f9b-4344-99bc-39bc2c8c88cb"
           (reference "#PWR07") (unit 1)
@@
         )
       )
-      (project "stm32_hotswap_chiffre"
+      (project "stm32_chiffre_36keys"
         (path "/ca0d59d2-7f9b-4344-99bc-39bc2c8c88cb"
           (reference "#PWR022") (unit 1)
@@
         )
       )
-      (project "stm32_hotswap_chiffre"
+      (project "stm32_chiffre_36keys"
         (path "/ca0d59d2-7f9b-4344-99bc-39bc2c8c88cb"
           (reference "C6") (unit 1)
@@
         )
       )
-      (project "stm32_hotswap_chiffre"
+      (project "stm32_chiffre_36keys"
         (path "/ca0d59d2-7f9b-4344-99bc-39bc2c8c88cb"
           (reference "C2") (unit 1)
@@
     (pin "1")
     (instances
-      (project "stm32_hotswap_chiffre"
+      (project "stm32_chiffre_36keys"
         (path "/ca0d59d2-7f9b-4344-99bc-39bc2c8c88cb"
           (reference "#PWR010") (unit 1)
@@
     (pin "2")
     (instances
-      (project "stm32_hotswap_chiffre"
+      (project "stm32_chiffre_36keys"
         (path "/ca0d59d2-7f9b-4344-99bc-39bc2c8c88cb"
           (reference "F1") (unit 1)
@@
     (pin "4")
     (instances
-      (project "stm32_hotswap_chiffre"
+      (project "stm32_chiffre_36keys"
         (path "/ca0d59d2-7f9b-4344-99bc-39bc2c8c88cb"
           (reference "J2") (unit 1)
@@
     (pin "1")
     (instances
-      (project "stm32_hotswap_chiffre"
+      (project "stm32_chiffre_36keys"
         (path "/ca0d59d2-7f9b-4344-99bc-39bc2c8c88cb"
           (reference "#PWR013") (unit 1)
@@
         )
       )
-      (project "stm32_hotswap_chiffre"
+      (project "stm32_chiffre_36keys"
         (path "/ca0d59d2-7f9b-4344-99bc-39bc2c8c88cb"
           (reference "R1") (unit 1)
@@
     (pin "1")
     (instances
-      (project "stm32_hotswap_chiffre"
+      (project "stm32_chiffre_36keys"
         (path "/ca0d59d2-7f9b-4344-99bc-39bc2c8c88cb"
           (reference "#PWR06") (unit 1)
@@
         )
       )
-      (project "stm32_hotswap_chiffre"
+      (project "stm32_chiffre_36keys"
         (path "/ca0d59d2-7f9b-4344-99bc-39bc2c8c88cb"
           (reference "R3") (unit 1)
@@
         )
       )
-      (project "stm32_hotswap_chiffre"
+      (project "stm32_chiffre_36keys"
         (path "/ca0d59d2-7f9b-4344-99bc-39bc2c8c88cb"
           (reference "C8") (unit 1)
@@
     (pin "2")
     (instances
-      (project "stm32_hotswap_chiffre"
+      (project "stm32_chiffre_36keys"
         (path "/ca0d59d2-7f9b-4344-99bc-39bc2c8c88cb"
           (reference "R4") (unit 1)
@@
         )
       )
-      (project "stm32_hotswap_chiffre"
+      (project "stm32_chiffre_36keys"
         (path "/ca0d59d2-7f9b-4344-99bc-39bc2c8c88cb"
           (reference "C5") (unit 1)
@@
         )
       )
-      (project "stm32_hotswap_chiffre"
+      (project "stm32_chiffre_36keys"
         (path "/ca0d59d2-7f9b-4344-99bc-39bc2c8c88cb"
           (reference "C7") (unit 1)
@@
         )
       )
-      (project "stm32_hotswap_chiffre"
+      (project "stm32_chiffre_36keys"
         (path "/ca0d59d2-7f9b-4344-99bc-39bc2c8c88cb"
           (reference "SW37") (unit 1)
@@
     (pin "1")
     (instances
-      (project "stm32_hotswap_chiffre"
+      (project "stm32_chiffre_36keys"
         (path "/ca0d59d2-7f9b-4344-99bc-39bc2c8c88cb"
           (reference "#PWR017") (unit 1)
@@
         )
       )
-      (project "stm32_hotswap_chiffre"
+      (project "stm32_chiffre_36keys"
         (path "/ca0d59d2-7f9b-4344-99bc-39bc2c8c88cb"
           (reference "#PWR023") (unit 1)
@@
     )
     (instances
-      (project "stm32_hotswap_chiffre"
+      (project "stm32_chiffre_36keys"
         (path "/ca0d59d2-7f9b-4344-99bc-39bc2c8c88cb" (page "2"))
       )
@@
     )
     (instances
-      (project "stm32_hotswap_chiffre"
+      (project "stm32_chiffre_36keys"
         (path "/ca0d59d2-7f9b-4344-99bc-39bc2c8c88cb" (page "3"))
       )
